Commit message: make new model

File: amr_proto_diff_drive/description/common_properties.xacro (robot description, xacro)
@@ -2,39 +2,12 @@
 <robot xmlns:xacro="http://www.ros.org/wiki/xacro">
     <!-- MATERIAL DEFINITION -->
-    <material name="green">
-        <color rgba="0 0.6 0 1" />
+    <material name="orange">
+        <color rgba="0.8 0.4 0.0 1.0"/>
     </material>
-    <material name="grey">
-        <color rgba="0.7 0.7 0.7 1" />
+    <material name="black">
+        <color rgba="0 0 0 1.0"/>
     </material>
     <material name="white">
-        <color rgba="1 1 1 1" />
+        <color rgba="1 1 1 1.0"/>
     </material>
-    <xacro:macro name="box_inertia" params="m x y z o_xyz o_rpy">
-        <inertial>
-            <mass value="${m}" />
-            <origin xyz="${o_xyz}" rpy="${o_rpy}" />
-            <inertia ixx="${(m/12) * (z*z + y*y)}" ixy="0" ixz="0"
-                    iyy="${(m/12) * (x*x + z*z)}" iyz="0"
-                    izz="${(m/12) * (x*x + y*y)}" />
-        </inertial>
-    </xacro:macro>
-    <xacro:macro name="cylinder_inertia" params="m r l o_xyz o_rpy">
-        <inertial>
-            <mass value="${m}" />
-            <origin xyz="${o_xyz}" rpy="${o_rpy}"/>
-            <inertia    ixx="${(m/12)*(3*r*r+l*l)}" ixy="0" ixz="0"
-                        iyy="${(m/12)*(3*r*r+l*l)}" iyz="0"
-                        izz="${(m/2)*(r*r)}" />
-        </inertial>
-    </xacro:macro>
-    <xacro:macro name="sphere_inertia" params="m r o_xyz o_rpy">
-        <inertial>
-            <mass value="${m}" />
-            <origin xyz="${o_xyz}" rpy="${o_rpy}" />
-            <inertia    ixx="${(2/5)*m*r*r}" ixy="0" ixz="0"
-                        iyy="${(2/5)*m*r*r}" iyz="0"
-                        izz="${(2/5)*m*r*r}" />
-        </inertial>
-</xacro:macro>
 </robot>

File: amr_proto_diff_drive/description/mobile_base.xacro (robot description, xacro)
@@ -1,90 +1,127 @@
 <?xml version="1.0"?>
 <robot xmlns:xacro="http://www.ros.org/wiki/xacro">
-    <!--BASE FOOTPRINT  -->
   <link name="base_footprint"/>
-  <!-- BASE -->
-  <link name="base_link">
+  <!-- Base Link -->
+  <link name="chassis">
+    <collision>
+      <origin xyz="-0.151427 -0 0.5" rpy="0 0 0"/>
+      <geometry>
+        <box size="2.01142 1 0.568726"/>
+      </geometry>
+    </collision>
+    <visual>
+      <origin xyz="-0.151427 -0 0.5" rpy="0 0 0"/>
+      <geometry>
+        <box size="2.01142 1 0.568726"/>
+      </geometry>
+      <material name="orange"/>
+    </visual>
+    <inertial>
+      <origin xyz="-0.151427 -0 0.5" rpy="0 0 0"/>
+      <mass value="1.14395"/>
+      <inertia
+        ixx="0.126164"
+        ixy="0.0"
+        ixz="0.0"
+        iyy="0.416519"
+        iyz="0.0"
+        izz="0.481014"/>
+    </inertial>
+  </link>
+  <!-- left wheel Link -->
+  <link name="left_wheel">
+    <collision>
+      <geometry>
+        <sphere radius="0.3"/>
+      </geometry>
+    </collision>
     <visual>
       <geometry>
-        <box size="0.6 0.4 0.2"/>
+        <sphere radius="0.3"/>
       </geometry>
-      <origin xyz="0.0 0.0 0.1" rpy="0.0 0.0 0.0"/>
-      <material name="green"/>
+      <material name="black"/>
     </visual>
+    <inertial>
+      <mass value="2"/>
+      <inertia ixx="0.145833"
+               ixy="0.0"
+               ixz="0.0"
+               iyy="0.145833"
+               iyz="0.0"
+               izz="0.125"/>
+    </inertial>
+  </link>
+  <!-- right wheel Link -->
+  <link name="right_wheel">
     <collision>
-      <origin xyz="0.0 0.0 0.1" rpy="0.0 0.0 0.0"/>
       <geometry>
-        <box size="0.6 0.4 0.2"/>
+        <sphere radius="0.3"/>
       </geometry>
     </collision>
-    <xacro:box_inertia  m="5.0" x="0.6" y="0.4" z="0.2"
-                        o_xyz="0 0 0.1" o_rpy="0 0 0"/>
-  </link>
-  <!-- MACRO FOR WHEEL LINK -->
-  <xacro:macro name="wheel_link" params="prefix">
-    <link name="${prefix}_wheel_link">
-      <visual>
-        <geometry>
-          <cylinder radius="0.1" length="0.05"/>
-        </geometry>
-        <origin xyz="0.0 0.0 0.0" rpy="1.571 0.0 0.0"/>
-        <material name="grey"/>
-      </visual>
-      <collision>
-        <origin xyz="0.0 0.0 0.0" rpy="0.0 0.0 0.0"/>
-        <geometry>
-          <sphere radius="0.1"/>
-        </geometry>
-      </collision>
-      <xacro:cylinder_inertia m="1.0" r="0.1" l="0.05"
-                              o_xyz="0 0 0" o_rpy="1.571 0 0" />
-    </link>
-  </xacro:macro>
-  <!-- CALL MACRO FOR RIGHT WHEEL AND LEFT WHEEL -->
-  <xacro:wheel_link prefix="left"/>
-  <xacro:wheel_link prefix="right"/>
-  <!-- CASTER WHEEL -->
-  <link name="caster_wheel_link">
     <visual>
       <geometry>
-        <sphere radius="0.05"/>
+        <sphere radius="0.3"/>
       </geometry>
-      <origin xyz="0.0 0.0 0.0" rpy="0.0 0.0 0.0"/>
-      <material name="grey"/>
+      <material name="black"/>
     </visual>
+    <inertial>
+      <mass value="2"/>
+      <inertia ixx="0.145833"
+               ixy="0.0"
+               ixz="0.0"
+               iyy="0.145833"
+               iyz="0.0"
+               izz="0.125"/>
+      </inertial>
+  </link>
+  <!-- caster frontal wheel Link -->
+  <link name="caster">
     <collision>
-      <origin xyz="0.0 0.0 0.0" rpy="0.0 0.0 0.0"/>
       <geometry>
-        <sphere radius="0.05"/>
+        <sphere radius="0.2"/>
       </geometry>
     </collision>
-    <xacro:sphere_inertia m="0.5" r="0.05"
-                          o_xyz="0 0 0" o_rpy="0 0 0" />
+    <visual>
+      <geometry>
+        <sphere radius="0.2"/>
+      </geometry>
+      <material name="white"/>
+    </visual>
+    <inertial>
+      <origin xyz="-0.957138 -0 0.2" rpy="0 0 0"/>
+      <mass value="0.005"/>
+      <inertia
+        ixx="0.1"
+        ixy="0.0"
+        ixz="0.0"
+        iyy="0.1"
+        iyz="0.0"
+        izz="0.1"/>
+    </inertial>
   </link>
-  <!-- BASE-LEFT WHEEL JOINT -->
+  <!-- JOINT    -->
+  <joint name="base_footprint_joint" type="fixed">
+    <origin xyz="0 0 0" rpy="0 0 0"/>
+    <parent link="base_footprint"/>
+    <child link="chassis"/>
+  </joint>
+  <joint name="caster_joint" type="fixed">
+    <origin xyz="-0.957138 -0 0.2" rpy="0 0 0"/>
+    <parent link="chassis"/>
+    <child link="caster"/>
+  </joint>
   <joint name="left_wheel_joint" type="continuous">
-    <origin xyz="-0.15 0.225 0.0" rpy="0.0 0.0 0.0"/>
-    <parent link="base_link"/>
-    <child link="left_wheel_link"/>
-    <axis xyz="0 1 0.0"/>
+    <origin xyz="0.554283 0.625029 0.3" rpy="-1.5707 0 0"/>
+    <parent link="chassis"/>
+    <child link="left_wheel"/>
+    <axis xyz="0 0 1"/>
+    <dynamics damping="0.2"/>
   </joint>
-  <!-- BASE-RIGHT WHEEL JOINT -->
   <joint name="right_wheel_joint" type="continuous">
-    <origin xyz="-0.15 -0.225 0.0" rpy="0.0 0.0 0.0"/>
-    <parent link="base_link"/>
-    <child link="right_wheel_link"/>
-    <axis xyz="0 1 0.0"/>
-  </joint>
-  <!-- BASE-CASTER JOINT  -->
-  <joint name="base_caster_wheel_joint" type="fixed">
-    <origin xyz="0.2 0.0 -0.05" rpy="0.0 0.0 0.0"/>
-    <parent link="base_link"/>
-    <child link="caster_wheel_link"/>
-  </joint>
-  <!-- BASE FOOTPRINT-BASE JOINT -->
-  <joint name="base_joint" type="fixed">
-    <origin xyz="0.0 0 0.1" rpy="0.0 0.0 0.0"/>
-    <parent link="base_footprint"/>
-    <child link="base_link"/>
+    <origin xyz="0.554283 -0.625029 0.3" rpy="-1.5707 0 0"/>
+    <parent link="chassis"/>
+    <child link="right_wheel"/>
+    <axis xyz="0 0 1"/>
+    <dynamics damping="0.2"/>
   </joint>
 </robot>

Commit message: new changes

File: amr_proto_diff_drive/description/common_properties.xacro (robot description, xacro)
@@ -2,6 +2,6 @@
 <robot xmlns:xacro="http://www.ros.org/wiki/xacro">
     <!-- MATERIAL DEFINITION -->
-    <material name="orange">
-        <color rgba="0.8 0.4 0.0 1.0"/>
+    <material name="green">
+    <color rgba="0.0 1.0 0.0 1.0"/>
     </material>
     <material name="black">
@@ -11,3 +11,18 @@
         <color rgba="1 1 1 1.0"/>
     </material>
+    <material name="blue">
+        <color rgba="0.0 0.0 0.8 1.0"/>
+    </material>
+    <material name="grey">
+        <color rgba="0.2 0.2 0.2 1.0"/>
+    </material>
+    <material name="orange">
+        <color rgba="${255/255} ${108/255} ${10/255} 1.0"/>
+    </material>
+    <material name="brown">
+        <color rgba="${222/255} ${207/255} ${195/255} 1.0"/>
+    </material>
+    <material name="red">
+        <color rgba="0.8 0.0 0.0 1.0"/>
+    </material>
 </robot>

File: amr_proto_diff_drive/description/lidar.xacro (robot description, xacro)
@@ -12,5 +12,5 @@
     <collision>
         <geometry>
-            <cylinder length="0.05" radius="0.1"/>
+            <cylinder length="0.2" radius="0.1"/>
         </geometry>
     </collision>
@@ -22,5 +22,5 @@
     <!-- BASE-LIDAR JOINT  -->
     <joint name="base_lidar_joint" type="fixed">
-        <origin xyz="0.26 0 0.23" rpy="0.0 0.0 0.0"/>
+        <origin xyz="0.3 0 0.8" rpy="0.0 0.0 0.0"/>
         <parent link="chassis"/>
         <child link="lidar"/>
@@ -51,5 +51,5 @@
                 <range>
                     <min>0.3</min>
-                    <max>12.0</max>
+                    <max>10.0</max>
                     <resolution>0.01</resolution>
                 </range>

File: amr_proto_diff_drive/description/mobile_base.xacro (robot description, xacro)
@@ -15,5 +15,5 @@
         <box size="2.01142 1 0.568726"/>
       </geometry>
-      <material name="orange"/>
+      <material name="red"/>
     </visual>
     <inertial>
@@ -100,4 +100,33 @@
     </inertial>
   </link>
+  <!-- caster rear wheel Link -->
+  <link name="caster_rear">
+    <collision>
+      <geometry>
+        <sphere radius="0.2"/>
+      </geometry>
+    </collision>
+    <visual>
+      <geometry>
+        <sphere radius="0.2"/>
+      </geometry>
+      <material name="white"/>
+    </visual>
+    <inertial>
+      <origin xyz="-0.957138 -0 0.2" rpy="0 0 0"/>
+      <mass value="0.005"/>
+      <inertia
+        ixx="0.1"
+        ixy="0.0"
+        ixz="0.0"
+        iyy="0.1"
+        iyz="0.0"
+        izz="0.1"/>
+    </inertial>
+  </link>
+  <gazebo reference="caster">
+      <mu1 value="0.001"/>
+      <mu2 value="0.001"/>
+  </gazebo>
   <!-- JOINT    -->
   <joint name="base_footprint_joint" type="fixed">
@@ -111,6 +140,11 @@
     <child link="caster"/>
   </joint>
+  <joint name="caster_joint_rear" type="fixed">
+    <origin xyz="0.4 -0 0.2" rpy="0 0 0"/>
+    <parent link="chassis"/>
+    <child link="caster_rear"/>
+  </joint>
   <joint name="left_wheel_joint" type="continuous">
-    <origin xyz="0.554283 0.625029 0.3" rpy="-1.5707 0 0"/>
+    <origin xyz="-0.0 0.625029 0.2" rpy="-1.5707 0 0"/>
     <parent link="chassis"/>
     <child link="left_wheel"/>
@@ -119,5 +153,5 @@
   </joint>
   <joint name="right_wheel_joint" type="continuous">
-    <origin xyz="0.554283 -0.625029 0.3" rpy="-1.5707 0 0"/>
+    <origin xyz="-0.0 -0.625029 0.2" rpy="-1.5707 0 0"/>
     <parent link="chassis"/>
     <child link="right_wheel"/>

File: amr_proto_diff_drive/description/robot_main.xacro (robot description, xacro)
@@ -3,4 +3,5 @@
     <xacro:include filename="common_properties.xacro"/>
     <!-- <xacro:include filename="mobile_base_stl.xacro"/> -->
+    <!-- <xacro:include filename="plugin_control.xacro"/> -->
     <xacro:include filename="mobile_base.xacro"/>
     <xacro:include filename="ros2_control.xacro"/>

File: amr_proto_diff_drive/description/ros2_control.xacro (robot description, xacro)
@@ -16,6 +16,6 @@
         <joint name="right_wheel_joint">
         <command_interface name="velocity">
-            <param name="min">-10</param>
-            <param name="max">10</param>
+            <param name="min">-1</param>
+            <param name="max">1</param>
         </command_interface>
         <state_interface name="position"/>
