Commit message: using gzebo classic

File: amr_proto_diff_drive/description/lidar.xacro (robot description, xacro)
@@ -28,38 +28,29 @@
     <!-- GAZEBO SIMULATED SENSOR LIDAR-->
     <gazebo reference="lidar">
-        <sensor type="gpu_lidar" name="lidar">
-            <always_on>true</always_on>
-            <enable_metrics>true</enable_metrics>
+        <!-- <material>Gazebo/Black</material> -->
+        <sensor name="laser" type="ray">
             <pose> 0 0 0 0 0 0 </pose>
-            <visualize>true</visualize>
-            <update_rate>30</update_rate>
+            <visualize>false</visualize>
+            <update_rate>10</update_rate>
             <ray>
                 <scan>
                     <horizontal>
-                        <resolution>1</resolution>
                         <samples>360</samples>
-                        <min_angle>-3.14159</min_angle>
-                        <max_angle>3.14159</max_angle>
+                        <min_angle>-3.14</min_angle>
+                        <max_angle>3.14</max_angle>
                     </horizontal>
-                    <vertical>
-                        <samples>1</samples>
-                        <resolution>0.01</resolution>
-                        <min_angle>0</min_angle>
-                        <max_angle>0</max_angle>
-                    </vertical>
                 </scan>
                 <range>
                     <min>0.3</min>
-                    <max>12.0</max>
-                    <resolution>0.01</resolution>
+                    <max>12</max>
                 </range>
-                <noise>
-                    <type>gaussian</type>
-                    <mean>0.0</mean>
-                    <stddev>0.01</stddev>
-                </noise>
             </ray>
-            <topic>scan</topic>
-            <gz_frame_id>lidar</gz_frame_id>
+            <plugin name="laser_controller" filename="libgazebo_ros_ray_sensor.so">
+                <ros>
+                    <argument>~/out:=scan</argument>
+                </ros>
+                <output_type>sensor_msgs/LaserScan</output_type>
+                <frame_name>lidar</frame_name>
+            </plugin>
         </sensor>
     </gazebo>

File: amr_proto_diff_drive/description/mobile_base.xacro (robot description, xacro)
@@ -44,4 +44,14 @@
   <xacro:wheel_link prefix="left"/>
   <xacro:wheel_link prefix="right"/>
+  <gazebo reference="left_wheel">
+      <material>Gazebo/Black</material>
+      <mu1 value="1.0"/>
+      <mu2 value="1.0"/>
+  </gazebo>
+  <gazebo reference="right_wheel">
+      <material>Gazebo/Black</material>
+      <mu1 value="1.0"/>
+      <mu2 value="1.0"/>
+  </gazebo>
   <!-- CASTER WHEEL -->
   <link name="caster_wheel_link">
@@ -62,4 +72,8 @@
                           o_xyz="0 0 0" o_rpy="0 0 0" />
   </link>
+  <gazebo reference="caster_wheel">
+      <mu1 value="0.001"/>
+      <mu2 value="0.001"/>
+  </gazebo>
   <!-- BASE-LEFT WHEEL JOINT -->
   <joint name="left_wheel_joint" type="continuous">

File: amr_proto_diff_drive/description/robot_main.xacro (robot description, xacro)
@@ -2,5 +2,5 @@
 <robot xmlns:xacro="http://www.ros.org/wiki/xacro" name="diff_drive=">
     <xacro:include filename="common_properties.xacro"/>
-    <!-- <xacro:include filename="mobile_base_coll_iner_with_stl.xacro"/> -->
+    <!-- <xacro:include filename="plugin_control.xacro"/> -->
     <xacro:include filename="mobile_base.xacro"/>
     <xacro:include filename="ros2_control.xacro"/>

File: amr_proto_diff_drive/description/ros2_control.xacro (robot description, xacro)
@@ -1,32 +1,29 @@
 <?xml version="1.0"?>
 <robot xmlns:xacro="http://www.ros.org/wiki/xacro">
-    <xacro:arg name="namespace" default="" />
-    <ros2_control name="GazeboSimSystem" type="system">
+    <ros2_control name="GazeboSystem" type="system">
         <hardware>
-            <plugin>gz_ros2_control/GazeboSimSystem</plugin>
+            <plugin>gazebo_ros2_control/GazeboSystem</plugin>
         </hardware>
         <joint name="left_wheel_joint">
-        <command_interface name="velocity">
-            <param name="min">-1</param>
-            <param name="max">1</param>
-        </command_interface>
-        <state_interface name="position"/>
-        <state_interface name="velocity"/>
+            <command_interface name="velocity">
+                <param name="min">-10</param>
+                <param name="max">10</param>
+            </command_interface>
+            <state_interface name="position"/>
+            <state_interface name="velocity"/>
         </joint>
         <joint name="right_wheel_joint">
-        <command_interface name="velocity">
-            <param name="min">-10</param>
-            <param name="max">10</param>
-        </command_interface>
-        <state_interface name="position"/>
-        <state_interface name="velocity"/>
+            <command_interface name="velocity">
+                <param name="min">-10</param>
+                <param name="max">10</param>
+            </command_interface>
+            <state_interface name="position"/>
+            <state_interface name="velocity"/>
         </joint>
     </ros2_control>
     <gazebo>
-        <plugin filename="gz_ros2_control-system" name="gz_ros2_control::GazeboSimROS2ControlPlugin">
-        <ros>
-            <namespace>$(arg namespace)</namespace>
-        </ros>
-        <parameters>$(find amr_proto_diff_drive)/config/diff_drive_controller.yaml</parameters>
+        <plugin name="gazebo_ros2_control" filename="libgazebo_ros2_control.so">
+            <parameters>$(find amr_proto_diff_drive)/config/diff_drive_controller.yaml</parameters>
+            <!-- <parameters>$(find amr_proto_diff_drive)/config/ros2_control_sim.yaml</parameters> -->
         </plugin>
     </gazebo>

Commit message: adding desc robot with stl

File: amr_proto_diff_drive/description/lidar.xacro (robot description, xacro)
@@ -22,6 +22,6 @@
     <!-- BASE-LIDAR JOINT  -->
     <joint name="base_lidar_joint" type="fixed">
-        <origin xyz="0 0 0.225" rpy="0.0 0.0 0.0"/>
-        <parent link="base_link"/>
+        <origin xyz="0.26 0 0.23" rpy="0.0 0.0 0.0"/>
+        <parent link="chassis"/>
         <child link="lidar"/>
     </joint>

File: amr_proto_diff_drive/description/robot_main.xacro (robot description, xacro)
@@ -1,7 +1,7 @@
 <?xml version="1.0"?>
-<robot xmlns:xacro="http://www.ros.org/wiki/xacro" name="diff_drive=">
+<robot xmlns:xacro="http://www.ros.org/wiki/xacro" name="diff_drive">
     <xacro:include filename="common_properties.xacro"/>
-    <!-- <xacro:include filename="mobile_base_coll_iner_with_stl.xacro"/> -->
-    <xacro:include filename="mobile_base.xacro"/>
+    <xacro:include filename="mobile_base_stl.xacro"/>
+    <!-- <xacro:include filename="mobile_base.xacro"/> -->
     <xacro:include filename="ros2_control.xacro"/>
     <xacro:include filename="lidar.xacro"/>

Commit message: stl

File: amr_proto_diff_drive/description/lidar.xacro (robot description, xacro)
@@ -23,5 +23,5 @@
     <joint name="base_lidar_joint" type="fixed">
         <origin xyz="0 0 0.225" rpy="0.0 0.0 0.0"/>
-        <parent link="base_link"/>
+        <parent link="chassis"/>
         <child link="lidar"/>
     </joint>

File: amr_proto_diff_drive/description/robot_main.xacro (robot description, xacro)
@@ -3,4 +3,5 @@
     <xacro:include filename="common_properties.xacro"/>
     <!-- <xacro:include filename="plugin_control.xacro"/> -->
+    <xacro:include filename="mobile_base_stl.xacro"/>
     <xacro:include filename="mobile_base.xacro"/>
     <xacro:include filename="ros2_control.xacro"/>
