Commit message: 2nd push

File: amr_proto_diff_drive/description/mobile_base.xacro (robot description, xacro)
@@ -1,14 +1,5 @@
 <?xml version="1.0"?>
-<robot name="amr_robot_proto" xmlns:xacro="http://www.ros.org/wiki/xacro">
-  <!-- MATERIAL DEFINITION -->
-  <material name="grey">
-    <color rgba=" 0.7 0.7 0.7 1"/>
-  </material>
-  <material name="green">
-    <color rgba="0.0 0.6 0.0 1.0"/>
-  </material>
-  <material name="white">
-    <color rgba="1 1 1 1"/>
-  </material>
+<robot xmlns:xacro="http://www.ros.org/wiki/xacro">
+    <!--BASE FOOTPRINT  -->
   <link name="base_footprint"/>
   <!-- BASE -->
@@ -21,4 +12,12 @@
       <material name="green"/>
     </visual>
+    <collision>
+      <origin xyz="0.0 0.0 0.1" rpy="0.0 0.0 0.0"/>
+      <geometry>
+        <box size="0.6 0.4 0.2"/>
+      </geometry>
+    </collision>
+    <xacro:box_inertia  m="5.0" x="0.6" y="0.4" z="0.2"
+                        o_xyz="0 0 0.1" o_rpy="0 0 0"/>
   </link>
   <!-- LIDAR -->
@@ -42,4 +41,12 @@
         <material name="grey"/>
       </visual>
+      <collision>
+        <origin xyz="0.0 0.0 0.0" rpy="0.0 0.0 0.0"/>
+        <geometry>
+          <sphere radius="0.1"/>
+        </geometry>
+      </collision>
+      <xacro:cylinder_inertia m="1.0" r="0.1" l="0.05"
+                              o_xyz="0 0 0" o_rpy="1.571 0 0" />
     </link>
   </xacro:macro>
@@ -56,4 +63,12 @@
       <material name="grey"/>
     </visual>
+    <collision>
+      <origin xyz="0.0 0.0 0.0" rpy="0.0 0.0 0.0"/>
+      <geometry>
+        <sphere radius="0.05"/>
+      </geometry>
+    </collision>
+    <xacro:sphere_inertia m="0.5" r="0.05"
+                          o_xyz="0 0 0" o_rpy="0 0 0" />
   </link>
   <!-- BASE-LIDAR JOINT  -->
@@ -64,5 +79,5 @@
   </joint>
   <!-- BASE-LEFT WHEEL JOINT -->
-  <joint name="base_left_wheel_joint" type="continuous">
+  <joint name="left_wheel_joint" type="continuous">
     <origin xyz="-0.15 0.225 0.0" rpy="0.0 0.0 0.0"/>
     <parent link="base_link"/>
@@ -71,5 +86,5 @@
   </joint>
   <!-- BASE-RIGHT WHEEL JOINT -->
-  <joint name="base_right_wheel_joint" type="continuous">
+  <joint name="right_wheel_joint" type="continuous">
     <origin xyz="-0.15 -0.225 0.0" rpy="0.0 0.0 0.0"/>
     <parent link="base_link"/>
@@ -77,5 +92,5 @@
     <axis xyz="0 1 0.0"/>
   </joint>
-    <!-- BASE-CASTER JOINT  -->
+  <!-- BASE-CASTER JOINT  -->
   <joint name="base_caster_wheel_joint" type="fixed">
     <origin xyz="0.2 0.0 -0.05" rpy="0.0 0.0 0.0"/>
@@ -83,4 +98,5 @@
     <child link="caster_wheel_link"/>
   </joint>
+  <!-- BASE FOOTPRINT-BASE JOINT -->
   <joint name="base_joint" type="fixed">
     <origin xyz="0.0 0 0.1" rpy="0.0 0.0 0.0"/>

Commit message: add lidar in ignition

File: amr_proto_diff_drive/description/mobile_base.xacro (robot description, xacro)
@@ -20,14 +20,4 @@
     <xacro:box_inertia  m="5.0" x="0.6" y="0.4" z="0.2"
                         o_xyz="0 0 0.1" o_rpy="0 0 0"/>
-  </link>
-  <!-- LIDAR -->
-  <link name="lidar_link">
-    <visual>
-      <geometry>
-          <cylinder radius="0.1" length="0.05"/>
-      </geometry>
-      <origin xyz="0.0 0.0 0.0" rpy="0.0 0.0 0.0"/>
-      <material name="white"/>
-    </visual>
   </link>
   <!-- MACRO FOR WHEEL LINK -->
@@ -72,10 +62,4 @@
                           o_xyz="0 0 0" o_rpy="0 0 0" />
   </link>
-  <!-- BASE-LIDAR JOINT  -->
-  <joint name="base_lidar_joint" type="fixed">
-    <origin xyz="0 0 0.225" rpy="0.0 0.0 0.0"/>
-    <parent link="base_link"/>
-    <child link="lidar_link"/>
-  </joint>
   <!-- BASE-LEFT WHEEL JOINT -->
   <joint name="left_wheel_joint" type="continuous">

File: amr_proto_diff_drive/description/robot_main.xacro (robot description, xacro)
@@ -5,3 +5,4 @@
     <xacro:include filename="mobile_base.xacro"/>
     <xacro:include filename="ros2_control.xacro"/>
+    <xacro:include filename="lidar.xacro"/>
 </robot>

File: amr_proto_diff_drive/description/ros2_control.xacro (robot description, xacro)
@@ -16,6 +16,6 @@
         <joint name="right_wheel_joint">
         <command_interface name="velocity">
-            <param name="min">-1</param>
-            <param name="max">1</param>
+            <param name="min">-10</param>
+            <param name="max">10</param>
         </command_interface>
         <state_interface name="position"/>

Commit message: add

File: amr_proto_diff_drive/description/mobile_base.xacro (robot description, xacro)
@@ -4,5 +4,5 @@
   <link name="base_footprint"/>
   <!-- BASE -->
-  <link name="base_link">
+  <link name="chassis">
     <visual>
       <geometry>
@@ -79,5 +79,5 @@
   <joint name="left_wheel_joint" type="continuous">
     <origin xyz="-0.15 0.225 0.0" rpy="0.0 0.0 0.0"/>
-    <parent link="base_link"/>
+    <parent link="chassis"/>
     <child link="left_wheel_link"/>
     <axis xyz="0 1 0.0"/>
@@ -86,5 +86,5 @@
   <joint name="right_wheel_joint" type="continuous">
     <origin xyz="-0.15 -0.225 0.0" rpy="0.0 0.0 0.0"/>
-    <parent link="base_link"/>
+    <parent link="chassis"/>
     <child link="right_wheel_link"/>
     <axis xyz="0 1 0.0"/>
@@ -93,5 +93,5 @@
   <joint name="base_caster_wheel_joint" type="fixed">
     <origin xyz="0.2 0.0 -0.05" rpy="0.0 0.0 0.0"/>
-    <parent link="base_link"/>
+    <parent link="chassis"/>
     <child link="caster_wheel_link"/>
   </joint>
@@ -100,5 +100,5 @@
     <origin xyz="0.0 0 0.1" rpy="0.0 0.0 0.0"/>
     <parent link="base_footprint"/>
-    <child link="base_link"/>
+    <child link="chassis"/>
   </joint>
 </robot>

File: amr_proto_diff_drive/description/robot_main.xacro (robot description, xacro)
@@ -3,5 +3,5 @@
     <xacro:include filename="common_properties.xacro"/>
     <!-- <xacro:include filename="plugin_control.xacro"/> -->
-    <xacro:include filename="mobile_base_stl.xacro"/>
+    <!-- <xacro:include filename="mobile_base_stl.xacro"/> -->
     <xacro:include filename="mobile_base.xacro"/>
     <xacro:include filename="ros2_control.xacro"/>
